File: Hardware/InterfaceModule/BidirectionalSwitch.kicad_sch (KiCad schematic)
At the start: 8 parts

Commit message: Picked some footprints for most connectors
Parts:
- gave numbers to parts that had none: 8
Changed lines of the file:
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@@
   (symbol (lib_id "Device:Q_PMOS_DGS") (at 163.83 66.04 270) (mirror x) (unit 1)
     (in_bom yes) (on_board yes) (fields_autoplaced)
-    (property "Reference" "Q?" (id 0) (at 163.83 57.6285 90))
+    (property "Reference" "Q2" (id 0) (at 163.83 57.6285 90))
     (property "Value" "Q_PMOS_DGS" (id 1) (at 163.83 60.4036 90))
     (property "Footprint" "" (id 2) (at 166.37 60.96 0)
@@
   (symbol (lib_id "power:GND") (at 143.51 99.06 0) (unit 1)
     (in_bom yes) (on_board yes) (fields_autoplaced)
-    (property "Reference" "#PWR?" (id 0) (at 143.51 105.41 0)
+    (property "Reference" "#PWR016" (id 0) (at 143.51 105.41 0)
       (effects (font (size 1.27 1.27)) hide)
     )
@@
   (symbol (lib_id "Device:D") (at 162.56 50.165 0) (mirror y) (unit 1)
     (in_bom yes) (on_board yes) (fields_autoplaced)
-    (property "Reference" "D?" (id 0) (at 162.56 44.9285 0))
+    (property "Reference" "D2" (id 0) (at 162.56 44.9285 0))
     (property "Value" "D" (id 1) (at 162.56 47.7036 0))
     (property "Footprint" "" (id 2) (at 162.56 50.165 0)
@@
   (symbol (lib_id "Device:R_US") (at 149.86 69.85 0) (unit 1)
     (in_bom yes) (on_board yes) (fields_autoplaced)
-    (property "Reference" "R?" (id 0) (at 151.511 68.9415 0)
+    (property "Reference" "R5" (id 0) (at 151.511 68.9415 0)
       (effects (font (size 1.27 1.27)) (justify left))
     )
@@
   (symbol (lib_id "Device:Q_PMOS_DGS") (at 123.825 66.04 90) (unit 1)
     (in_bom yes) (on_board yes) (fields_autoplaced)
-    (property "Reference" "Q?" (id 0) (at 123.825 57.6285 90))
+    (property "Reference" "Q1" (id 0) (at 123.825 57.6285 90))
     (property "Value" "Q_PMOS_DGS" (id 1) (at 123.825 60.4036 90))
     (property "Footprint" "" (id 2) (at 121.285 60.96 0)
@@
   (symbol (lib_id "Device:D") (at 125.095 50.165 0) (unit 1)
     (in_bom yes) (on_board yes) (fields_autoplaced)
-    (property "Reference" "D?" (id 0) (at 125.095 44.9285 0))
+    (property "Reference" "D1" (id 0) (at 125.095 44.9285 0))
     (property "Value" "D" (id 1) (at 125.095 47.7036 0))
     (property "Footprint" "" (id 2) (at 125.095 50.165 0)
@@
   (symbol (lib_id "Device:C") (at 137.16 69.85 0) (unit 1)
     (in_bom yes) (on_board yes) (fields_autoplaced)
-    (property "Reference" "C?" (id 0) (at 140.081 68.9415 0)
+    (property "Reference" "C1" (id 0) (at 140.081 68.9415 0)
       (effects (font (size 1.27 1.27)) (justify left))
     )
@@
   (symbol (lib_id "Device:Q_NMOS_DGS") (at 140.97 91.44 0) (unit 1)
     (in_bom yes) (on_board yes) (fields_autoplaced)
-    (property "Reference" "Q?" (id 0) (at 146.177 90.5315 0)
+    (property "Reference" "Q3" (id 0) (at 146.177 90.5315 0)
       (effects (font (size 1.27 1.27)) (justify left))
     )
@@
   (symbol (lib_id "Device:R_US") (at 143.51 80.01 0) (unit 1)
     (in_bom yes) (on_board yes) (fields_autoplaced)
-    (property "Reference" "R?" (id 0) (at 145.161 79.1015 0)
+    (property "Reference" "R6" (id 0) (at 145.161 79.1015 0)
       (effects (font (size 1.27 1.27)) (justify left))
     )
