File: Hardware/InterfaceModule/GPS.kicad_sch (KiCad schematic)
At the start: 0 parts

Commit message: Connections for data ports, gps, improved mic connections
Connections:
- no-connect marks 0 -> 1
Changed lines of the file:
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@@
 (kicad_sch (version 20211123) (generator eeschema)
   (paper "A4")
+  (junction (at 142.875 106.045) (diameter 0) (color 0 0 0 0)
+  )
+  (junction (at 131.445 95.885) (diameter 0) (color 0 0 0 0)
+  )
+  (no_connect (at 131.445 80.01))
+  (bus_entry (at 92.71 108.585) (size 2.54 -2.54)
+    (stroke (width 0) (type default) (color 0 0 0 0))
+  )
+  (bus_entry (at 92.71 103.505) (size 2.54 -2.54)
+    (stroke (width 0) (type default) (color 0 0 0 0))
+  )
+  (bus_entry (at 92.71 98.425) (size 2.54 -2.54)
+    (stroke (width 0) (type default) (color 0 0 0 0))
+  )
+  (bus_entry (at 183.515 103.505) (size -2.54 -2.54)
+    (stroke (width 0) (type default) (color 0 0 0 0))
+  )
+  (bus_entry (at 102.235 72.39) (size 2.54 2.54)
+    (stroke (width 0) (type default) (color 0 0 0 0))
+  )
+  (bus_entry (at 102.235 82.55) (size 2.54 2.54)
+    (stroke (width 0) (type default) (color 0 0 0 0))
+  )
+  (bus_entry (at 183.515 98.425) (size -2.54 -2.54)
+    (stroke (width 0) (type default) (color 0 0 0 0))
+  )
+  (bus_entry (at 183.515 108.585) (size -2.54 -2.54)
+    (stroke (width 0) (type default) (color 0 0 0 0))
+  )
+  (bus_entry (at 102.235 77.47) (size 2.54 2.54)
+    (stroke (width 0) (type default) (color 0 0 0 0))
+  )
+  (wire (pts (xy 104.775 74.93) (xy 142.875 74.93))
+    (stroke (width 0) (type default) (color 0 0 0 0))
+  )
+  (bus (pts (xy 92.71 103.505) (xy 92.71 98.425))
+    (stroke (width 0) (type default) (color 0 0 0 0))
+  )
+  (bus (pts (xy 102.235 72.39) (xy 102.235 77.47))
+    (stroke (width 0) (type default) (color 0 0 0 0))
+  )
+  (wire (pts (xy 131.445 95.885) (xy 180.975 95.885))
+    (stroke (width 0) (type default) (color 0 0 0 0))
+  )
+  (bus (pts (xy 196.215 108.585) (xy 183.515 108.585))
+    (stroke (width 0) (type default) (color 0 0 0 0))
+  )
+  (wire (pts (xy 104.775 80.01) (xy 131.445 80.01))
+    (stroke (width 0) (type default) (color 0 0 0 0))
+  )
+  (wire (pts (xy 95.25 100.965) (xy 180.975 100.965))
+    (stroke (width 0) (type default) (color 0 0 0 0))
+  )
+  (bus (pts (xy 183.515 108.585) (xy 183.515 103.505))
+    (stroke (width 0) (type default) (color 0 0 0 0))
+  )
+  (bus (pts (xy 183.515 103.505) (xy 183.515 98.425))
+    (stroke (width 0) (type default) (color 0 0 0 0))
+  )
+  (wire (pts (xy 142.875 74.93) (xy 142.875 106.045))
+    (stroke (width 0) (type default) (color 0 0 0 0))
+  )
+  (bus (pts (xy 102.235 77.47) (xy 102.235 82.55))
+    (stroke (width 0) (type default) (color 0 0 0 0))
+  )
+  (wire (pts (xy 104.775 85.09) (xy 131.445 85.09))
+    (stroke (width 0) (type default) (color 0 0 0 0))
+  )
+  (bus (pts (xy 92.71 108.585) (xy 92.71 103.505))
+    (stroke (width 0) (type default) (color 0 0 0 0))
+  )
+  (wire (pts (xy 95.25 95.885) (xy 131.445 95.885))
+    (stroke (width 0) (type default) (color 0 0 0 0))
+  )
+  (wire (pts (xy 95.25 106.045) (xy 142.875 106.045))
+    (stroke (width 0) (type default) (color 0 0 0 0))
+  )
+  (wire (pts (xy 131.445 85.09) (xy 131.445 95.885))
+    (stroke (width 0) (type default) (color 0 0 0 0))
+  )
+  (wire (pts (xy 142.875 106.045) (xy 180.975 106.045))
+    (stroke (width 0) (type default) (color 0 0 0 0))
+  )
+  (bus (pts (xy 89.535 72.39) (xy 102.235 72.39))
+    (stroke (width 0) (type default) (color 0 0 0 0))
+  )
+  (bus (pts (xy 80.01 108.585) (xy 92.71 108.585))
+    (stroke (width 0) (type default) (color 0 0 0 0))
+  )
+  (label "D-700_GPS.GPS_OUT" (at 104.775 80.01 0)
+    (effects (font (size 1.27 1.27)) (justify left bottom))
+  )
+  (label "EXTERNAL_GPS_OUT.GPS_IN" (at 180.975 100.965 180)
+    (effects (font (size 1.27 1.27)) (justify right bottom))
+  )
+  (label "EXTERNAL_GPS_IN.GPS_IN" (at 95.25 95.885 0)
+    (effects (font (size 1.27 1.27)) (justify left bottom))
+  )
+  (label "EXTERNAL_GPS_OUT.GPS_OUT" (at 180.975 95.885 180)
+    (effects (font (size 1.27 1.27)) (justify right bottom))
+  )
+  (label "D-700_GPS.GPS_IN" (at 104.775 85.09 0)
+    (effects (font (size 1.27 1.27)) (justify left bottom))
+  )
+  (label "D-700_GPS.GPS_GND" (at 104.775 74.93 0)
+    (effects (font (size 1.27 1.27)) (justify left bottom))
+  )
+  (label "EXTERNAL_GPS_IN.GPS_GND" (at 95.25 106.045 0)
+    (effects (font (size 1.27 1.27)) (justify left bottom))
+  )
+  (label "EXTERNAL_GPS_IN.GPS_OUT" (at 95.25 100.965 0)
+    (effects (font (size 1.27 1.27)) (justify left bottom))
+  )
+  (label "EXTERNAL_GPS_OUT.GPS_GND" (at 180.975 106.045 180)
+    (effects (font (size 1.27 1.27)) (justify right bottom))
+  )
+  (hierarchical_label "EXTERNAL_GPS_OUT{GPS_GND GPS_OUT GPS_IN}" (shape input) (at 196.215 108.585 0)
+    (effects (font (size 1.27 1.27)) (justify left))
+  )
+  (hierarchical_label "EXTERNAL_GPS_IN{GPS_GND GPS_OUT GPS_IN}" (shape input) (at 80.01 108.585 180)
+    (effects (font (size 1.27 1.27)) (justify right))
+  )
+  (hierarchical_label "D-700_GPS{GPS_GND GPS_OUT GPS_IN}" (shape input) (at 89.535 72.39 180)
+    (effects (font (size 1.27 1.27)) (justify right))
+  )
 )
