File: Hardware/AudioPanel/Planning/COM_DATA_Switching.kicad_sch (KiCad schematic)
At the start: 22 parts, among them J27 Debug Header, SW15 ~{RESET}, SW16 ~{RESET}, SW9 ~{RESET}, U104 MCP23017_ML, U42 ATtiny3227-M, U45 MCP23017_ML, U96 MCP23017_ML, Y7 20MHz

Commit message: More things
Connections:
- net 480_DATA_.SQCIN renamed 480_DATA.SQCIN
- net 700_DATA_.SQCIN renamed 700_DATA.SQCIN
- net 710_DATA_.SQCIN renamed 710_DATA.SQCIN
- net EXTRA_DATA_.SQCIN renamed EXTRA_DATA.SQCIN
Changed lines of the file:
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@@
 		)
 	)
-	(label "700_DATA_.SQCIN"
+	(label "700_DATA.SQCIN"
 		(at 135.89 207.01 0)
 		(effects
@@
 		)
 	)
-	(label "700_DATA_.SQCIN"
+	(label "700_DATA.SQCIN"
 		(at 53.34 193.04 180)
 		(effects
@@
 		)
 	)
-	(label "710_DATA_.SQCIN"
+	(label "710_DATA.SQCIN"
 		(at 135.89 224.79 0)
 		(effects
@@
 		)
 	)
-	(label "480_DATA_.SQCIN"
+	(label "480_DATA.SQCIN"
 		(at 53.34 161.29 180)
 		(effects
@@
 		)
 	)
-	(label "710_DATA_.SQCIN"
+	(label "710_DATA.SQCIN"
 		(at 53.34 224.79 180)
 		(effects
@@
 		)
 	)
-	(label "EXTRA_DATA_.SQCIN"
+	(label "EXTRA_DATA.SQCIN"
 		(at 53.34 256.54 180)
 		(effects
@@
 		)
 	)
-	(label "480_DATA_.SQCIN"
+	(label "480_DATA.SQCIN"
 		(at 135.89 201.93 0)
 		(effects
@@
 		)
 	)
-	(label "EXTRA_DATA_.SQCIN"
+	(label "EXTRA_DATA.SQCIN"
 		(at 135.89 229.87 0)
 		(effects
