File: Hardware/AudioPanel/Dev Modules/Kenwood Microphone Switcher/SIPO.kicad_sch (KiCad schematic)
At the start: 13 parts, among them U1201 SN74LV595ARGYR, U1202 SN74LV595ARGYR, U1203 SN74LV595ARGYR, U1204 SN74LV595ARGYR, U1205 SN74LV595ARGYR, U1206 SN74LV595ARGYR

Commit message: Added labeling and organized pages
Other:
- company: (none) -> Thomas Francois - KX∅STL
- title: (none) -> Kenwood Handset Switcher - SIPOs
Changed lines of the file:
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@@
 	(generator_version "9.0")
 	(paper "B")
+	(title_block
+		(title "Kenwood Handset Switcher - SIPOs")
+		(date "2025-07-11")
+		(rev "A")
+		(company "Thomas Francois - KX∅STL")
+	)
 	(text "595-F"
 		(exclude_from_sim no)
