File: Hardware/AudioPanel/Dev Modules/DATA Switcher/Crosspoint_8x8_Partial_4066.kicad_sch (KiCad schematic)
At the start: 114 parts, among them U701 74HC4066BQ, U702 74HC4066BQ, U703 74HC4066BQ, U704 74HC4066BQ, U705 74HC4066BQ, U706 74HC4066BQ, U707 74HC4066BQ, U708 74HC4066BQ, U709 74HC4066BQ, U710 74HC4066BQ, U711 74HC4066BQ, U712 74HC4066BQ, U713 74HC4066BQ, U714 74HC4066BQ

Commit message: DATA switcher put together
Parts:
- renumbered C701 to C1001, C702 to C1002, C703 to C1003, C704 to C1004, C705 to C1005, C706 to C1006, C707 to C1007, C708 to C1008, C709 to C1009, C710 to C1010, C711 to C1011, C712 to C1012, C713 to C1013, C714 to C1014, C715 to C1015, C716 to C1016, D701 to D1001, D729 to D1002, D702 to D1003, D730 to D1004, D703 to D1005, D731 to D1006, D704 to D1007, D732 to D1008, D705 to D1009, D733 to D1010, D706 to D1011, D734 to D1012, D707 to D1013, D735 to D1014, D708 to D1015, D736 to D1016, D709 to D1017, D737 to D1018, D710 to D1019, D738 to D1020, D711 to D1021, D739 to D1022, D712 to D1023, D740 to D1024, D713 to D1025, D741 to D1026, D714 to D1027, D742 to D1028, D715 to D1029, D743 to D1030, D716 to D1031, D744 to D1032, D717 to D1033, D745 to D1034, D718 to D1035, D746 to D1036, D719 to D1037, D747 to D1038, D720 to D1039, D748 to D1040, D721 to D1041, D749 to D1042, D722 to D1043, D750 to D1044, D723 to D1045, D751 to D1046, D724 to D1047, D752 to D1048, D725 to D1049, D753 to D1050, D726 to D1051, D754 to D1052, D727 to D1053, D755 to D1054, D728 to D1055, D756 to D1056, RN715 to RN1001, RN722 to RN1002, RN701 to RN1003, RN702 to RN1004, RN716 to RN1005, RN723 to RN1006, RN703 to RN1007, RN704 to RN1008, RN717 to RN1009, RN724 to RN1010, RN705 to RN1011, RN706 to RN1012, RN707 to RN1013, RN718 to RN1014, RN725 to RN1015, RN708 to RN1016, RN709 to RN1017, RN719 to RN1018, RN726 to RN1019, RN710 to RN1020, RN711 to RN1021, RN712 to RN1022, RN720 to RN1023, RN727 to RN1024, RN713 to RN1025, RN714 to RN1026, RN721 to RN1027, RN728 to RN1028, U707 to U1001, U702 to U1002, U714 to U1003, U703 to U1004, U704 to U1005, U705 to U1006, U706 to U1007, U701 to U1008, U708 to U1009, U713 to U1010, U709 to U1011, U712 to U1012, U710 to U1013, U711 to U1014
