File: Hardware/AudioPanel/Dev Modules/DATA Switcher/SIPO_16bit.kicad_sch (KiCad schematic)
At the start: 7 parts, among them U1001 SN74LV595ARGYR, U1002 SN74LV595ARGYR, U1003 SN74LV595ARGYR

Commit message: Many tweaks
Parts:
- removed U1003: SN74LV595ARGYR, Libraries:RGY16_2P55X2P05, symbol 74xx:74HC595
- renumbered C1001 to C901, C1002 to C902, C1003 to C903, C1008 to C904, U1001 to U901, U1002 to U902
Connections:
- net 595_B-C is gone; now on net SERIAL_OUT: U902.9 (QH')
- net +5V_IN: now also U901.16 (VCC)
- net A1: now also U901.4 (QE); no longer U901.15 (QA)
- net A2: now also U901.5 (QF); no longer U901.1 (QB)
- net A3: now also U901.6 (QG); no longer U901.2 (QC)
- net B0: now also U901.7 (QH); no longer U901.3 (QD)
- net B2: now also U902.15 (QA); no longer U901.4 (QE)
- net B3: now also U902.1 (QB); no longer U901.5 (QF)
- net C0: now also U902.2 (QC); no longer U901.6 (QG)
- net C1: now also U902.3 (QD); no longer U901.7 (QH)
- net C3: now also U902.4 (QE); no longer U902.15 (QA)
- net D0: now also U902.5 (QF); no longer U902.1 (QB)
- net D1: now also U902.6 (QG); no longer U902.2 (QC)
- net D2: now also U902.7 (QH); no longer U902.3 (QD)
- new net BIT_0: U901.15 (QA)
- new net BIT_1: U901.1 (QB)
- new net BIT_2: U901.2 (QC)
- new net BIT_3: U901.3 (QD)
Other:
- note removed: "595-C"
